Commit message: add project report

File: urdf/my_bot.xacro (robot description, xacro)
@@ -1,5 +1,5 @@
 <?xml version='1.0'?>
 <robot name="udacity_bot" xmlns:xacro="http://www.ros.org/wiki/xacro">
-  <xacro:include filename="$(find udacity_bot)/urdf/udacity_bot.gazebo" />
+  <xacro:include filename="$(find udacity_bot)/urdf/my_bot.gazebo" />
   <link name="robot_footprint"></link>
   <joint name="robot_footprint_joint" type="fixed">
@@ -53,26 +53,4 @@
       </geometry>
     </visual>
-    <collision name='front_caster_collision'>
-      <origin xyz="0.075 0 -0.025" rpy=" 0 0 0"/>
-      <geometry>
-        <sphere radius="0.025"/>
-      </geometry>
-      <surface>
-        <friction>
-          <ode>
-            <mu>0</mu>
-            <mu2>0</mu2>
-            <slip1>.9</slip1>
-            <slip2>1.0</slip2>
-          </ode>
-        </friction>
-      </surface>
-    </collision>
-    <visual name='front_caster_visual'>
-      <origin xyz=".075 0 -.025" rpy=" 0 0 0"/>
-      <geometry>
-        <sphere radius=".025"/>
-      </geometry>
-    </visual>
   </link>
   <link name="left_wheel">
@@ -92,5 +70,5 @@
       </geometry>
     </collision>
-    <visual name='chassis_visual'>
+    <visual name='lwheel_visual'>
       <origin xyz="0 0 0" rpy="0 1.5707 1.5707"/>
       <geometry>
@@ -100,5 +78,5 @@
   </link>
   <joint type="continuous" name="left_wheel_hinge">
-    <origin xyz="0 0.075 0" rpy="0 0 0"/>
+    <origin xyz="0.05 0.075 0" rpy="0 0 0"/>
     <child link="left_wheel"/>
     <parent link="chassis"/>
@@ -123,5 +101,5 @@
       </geometry>
     </collision>
-    <visual name='chassis_visual'>
+    <visual name='rwheel_visual'>
       <origin xyz="0 0 0" rpy="0 1.5707 1.5707"/>
       <geometry>
@@ -131,5 +109,5 @@
   </link>
   <joint type="continuous" name="right_wheel_hinge">
-    <origin xyz="0 -0.075 0" rpy="0 0 0"/>
+    <origin xyz="0.05 -0.075 0" rpy="0 0 0"/>
     <child link="right_wheel"/>
     <parent link="chassis"/>
@@ -155,8 +133,8 @@
       </geometry>
     </collision>
-    <visual name='chassis_visual'>
+    <visual name='cam_visual'>
       <origin xyz="0 0 0" rpy="0 0 0"/>
       <geometry>
-        <box size="0.025 0.025 0.025"/>
+              <mesh filename="package://udacity_bot/meshes/realsense.dae"/>
       </geometry>
     </visual>
@@ -185,5 +163,5 @@
       </geometry>
     </collision>
-    <visual name='chassis_visual'>
+    <visual name='laser_visual'>
       <origin xyz="0 0 0" rpy="0 0 0"/>
       <geometry>

File: urdf/udacity_bot.xacro (robot description, xacro)
@@ -184,5 +184,5 @@
       </geometry>
     </collision>
-    <visual name='camera_visual'>
+    <visual name='chassis_visual'>
       <origin xyz="0.0 0 0.0" rpy=" 0 0 0"/>
       <geometry>
